File: HW/BackBoard/purplewizard.kicad_pcb (KiCad board)
At the start: 2 copper layers, 92.5 x 151 mm, 146 parts, among them J1 3.3V, J10 SPKR-, J11 JTAG, J12 TagConnect, J13 Minibadge Expansion, J14 Battery, J15 USB_C_Receptacle_USB2.0, J16 Conn_01x50, J17 Board to Board, J18 Micro_SD_Card, J19 UPDI Programming, J2 GND, J3 UART_TX, J4 UART_RX, J5 LCD_SCK, J6 LCD_MOSI, J8 LCD_RS, J9 SPKR+, Q1 FDN360P, SW1 Power, SW10 TACTILE, SW11 TACTILE, SW12 TACTILE, SW13 TACTILE, SW14 TACTILE, SW15 TACTILE, SW16 TACTILE, SW17 TACTILE, SW18 SKRHABE010, SW19 SKRHABE010, SW2 TACTILE, SW3 TACTILE, SW4 TACTILE, SW5 TACTILE, SW6 TACTILE, SW7 TACTILE, SW8 TACTILE, SW9 TACTILE, U1 NAU8810, U2 SC189ZSKTRT, U3 BMD-340, U4 MCP73832-2-OT, U5 S25FL256S, U6 IS31FL3736, U7 ATtiny1617-M, X1 Badgelife_sao_connector_v169b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

Commit message: Backboard - Move LCD connector over .3mm for better fitment of ribbon - Fix audio chip missing exposed pad bond to ground - Remove nRESET signal from JTAG - Reuse freed pin above to run an interrupt line from the keyboard controller to the MCU to enable interrupt driven keyboard input.  Protos will have a hack-n-jump to be feature compatible - Enlarge mounting holes from 3mm to 3.2mm to allow for slightly sloppier fitments - Move traces and vias a little further away from top mounting holes as they are now being used for standoffs instead of just lanyard holes - Move vias from pads of ghosting diodes off to the side to prevent excess solder wicking - Modify UPDI programming pads to include vias for easier connection of programmer - Enlarged fiducials - Moved LCD CS from high to low - Added more breakout pads for the LCD on the back - Swapped to a PAM2305 voltage regulator - Hardwired the LCD LED to ground - Added some breakout for a couple of processor GPIO - Moved silk for speaker placement down a little - Added logo for PCBX Artboard - Remove mask over eyes
Parts:
- added C26: 10uF, Capacitor_SMD:C_0603_1608Metric, B.Cu at (147.6, 105.9)
- added G***: LOGO, common_fp:pcbx_logo, B.Cu at (171.1, 167.0)
- added J20: P1.06, TestPoint:TestPoint_Pad_1.5x1.5mm, B.Cu at (188.6, 137.5)
- added J21: P1.05, TestPoint:TestPoint_Pad_1.5x1.5mm, B.Cu at (188.6, 135.0)
- added J22: LCD_MISO, TestPoint:TestPoint_Pad_1.5x1.5mm, B.Cu at (143.6, 92.1)
- added J23: LCD_RD, TestPoint:TestPoint_Pad_1.5x1.5mm, B.Cu at (143.6, 97.1)
- added J24: LCD_TE, TestPoint:TestPoint_Pad_1.5x1.5mm, B.Cu at (143.6, 104.8)
- added J25: MOUT, TestPoint:TestPoint_Pad_1.5x1.5mm, B.Cu at (159.0, 68.1)
- added J26: MIC+, TestPoint:TestPoint_Pad_1.5x1.5mm, B.Cu at (177.3, 71.9)
- added J27: GND, TestPoint:TestPoint_Pad_1.5x1.5mm, B.Cu at (180.8, 71.9)
- added J7: P1.07, TestPoint:TestPoint_Pad_1.5x1.5mm, B.Cu at (188.6, 140.1)
- added JP1: SolderJumper_2_Bridged, Jumper:SolderJumper-2_P1.3mm_Bridged_RoundedPad1.0x1.5mm, B.Cu at (146.1, 97.9)
- added R17: 540k, Resistor_SMD:R_0603_1608Metric, B.Cu at (105.2, 154.1)
- added R18: 120k, Resistor_SMD:R_0603_1608Metric, B.Cu at (105.2, 157.3)
- D10: value LED -> ADD
- D11: value LED -> MEM1
- D12: value LED -> BIT64
- D13: value LED -> BIT4
- D14: value LED -> HAX
- D15: value LED -> SUB
- D16: value LED -> MEM2
- D17: value LED -> BIT32
- D18: value LED -> BIT2
- D19: value LED -> SD
- D20: value LED -> PAGE
- D21: value LED -> MEM3
- D22: value LED -> BIT16
- D23: value LED -> BIT1
- D5: value LED -> XOR
- D6: value LED -> MEM0
- D7: value LED -> BIT128
- D8: value LED -> BIT8
- D9: value LED -> USB
- FID1, FID2, FID3, FID4: footprint Fiducial:Fiducial_0.5mm_Mask1.5mm -> Fiducial:Fiducial_1mm_Mask2mm
- J8: value LCD_RS -> LCD_WR
- L1: value 1.0uH -> 4.7uH; footprint Inductor_SMD:L_Abracon_ASPI-3012S -> Inductor_SMD:L_0805_2012Metric
- U2: value SC189ZSKTRT -> PAM2305AABADJ
- U6: footprint Package_DFN_QFN:QFN-40-1EP_5x5mm_P0.4mm_EP3.6x3.6mm_ThermalVias -> lib_fp:QFN-40-1EP_5x5mm_P0.4mm_EP3.6x3.6mm_LargerThermalVias
- moved C25 17.1 mm to (147.7, 108.0), turned to 0 degrees
- moved FID4 14.5 mm to (181.4, 165.8)
- moved FID3 8.09 mm to (107.7, 79.0)
- moved J6 5.90 mm to (143.6, 94.6)
- moved C6 5.33 mm to (111.1, 154.3)
- moved J5 5.11 mm to (143.6, 102.2)
- moved J8 4.36 mm to (143.6, 99.7)
- moved J9 3.31 mm to (159.0, 64.7)
- moved J10 3.25 mm to (159.0, 61.3)
- moved C3 1.45 mm to (111.1, 157.6)
- moved U2 1.44 mm to (108.0, 156.0)
- moved R1 1.31 mm to (114.8, 153.2), turned to 180 degrees
- moved L1 0.53 mm to (108.9, 152.3), turned to 90 degrees
- moved J16 0.34 mm to (153.5, 98.2)
Connections:
- net LCD_RS renamed LCD_WR
- J11 pad 10: nRESET -> Net-(J11-Pad10)
- J12 pad 10: nRESET -> Net-(J12-Pad10)
- J16 pad 11: Net-(J16-Pad11) -> GND
- J16 pad 12: Net-(J16-Pad12) -> GND
- J16 pad 13: Net-(J16-Pad13) -> GND
- J16 pad 14: Net-(J16-Pad14) -> GND
- J16 pad 15: Net-(J16-Pad15) -> GND
- J16 pad 16: Net-(J16-Pad16) -> GND
- J16 pad 17: Net-(J16-Pad17) -> GND
- J16 pad 18: Net-(J16-Pad18) -> GND
- J16 pad 19: Net-(J16-Pad19) -> GND
- J16 pad 2: LCD_LED -> GND
- J16 pad 20: Net-(J16-Pad20) -> GND
- J16 pad 21: Net-(J16-Pad21) -> GND
- J16 pad 22: Net-(J16-Pad22) -> GND
- J16 pad 23: Net-(J16-Pad23) -> GND
- J16 pad 24: Net-(J16-Pad24) -> GND
- J16 pad 25: Net-(J16-Pad25) -> GND
- J16 pad 26: Net-(J16-Pad26) -> GND
- J16 pad 27: Net-(J16-Pad27) -> GND
- J16 pad 28: Net-(J16-Pad28) -> GND
- J16 pad 29: Net-(J16-Pad29) -> GND
- J16 pad 3: LCD_LED -> GND
- J16 pad 30: Net-(J16-Pad30) -> GND
- J16 pad 31: Net-(J16-Pad31) -> GND
- J16 pad 32: Net-(J16-Pad32) -> GND
- J16 pad 33: Net-(J16-Pad33) -> LCD_MISO
- J16 pad 35: Net-(J16-Pad35) -> LCD_RD
- J16 pad 38: +3V3 -> GND
- J16 pad 39: Net-(J16-Pad39) -> LCD_TE
- J16 pad 4: LCD_LED -> GND
- J16 pad 5: LCD_LED -> GND
- U1 pad 6: Net-(U1-Pad6) -> I2S_SDIN
- U2 pad 4: +3V3 -> Net-(R17-Pad1)
- U3 pad 12: LCD_LED -> I2S_SDIN
- U3 pad 39: nRESET -> KEY_INT
- U7 pad 22: Net-(U7-Pad22) -> KEY_INT
Routing:
- net I2S_SDIN: track 0.00 -> 98.2 mm, vias 0 -> 4
- net LCD_LED: track 85.6 -> 0.00 mm
- net KEY_INT: track 0.00 -> 64.9 mm, vias 0 -> 5
- net GND: track 217.0 -> 262.1 mm, vias 56 -> 62
- net nRESET: track 38.3 -> 0.00 mm, vias 2 -> 0
- net Net-(J26-Pad1): track 0.00 -> 18.4 mm, vias 0 -> 2
- net LCD_MISO: track 0.00 -> 17.5 mm
- net LCD_RD: track 0.00 -> 13.4 mm
- net Net-(J7-Pad1): track 0.00 -> 12.6 mm, vias 0 -> 2
- net Net-(J20-Pad1): track 0.00 -> 9.63 mm, vias 0 -> 2
- net SCL: track 286.8 -> 296.0 mm, vias 9 -> 8
- net LCD_TE: track 0.00 -> 8.23 mm
- net LCD_MOSI: track 68.8 -> 76.3 mm
- net Net-(J25-Pad1): track 0.00 -> 7.39 mm
- net SDA: track 281.3 -> 288.5 mm
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- added copper zone on B.Cu, net +BATT_SW
- added copper zone on F.Cu, net GND
Other:
- outline, holes or cut-outs redrawn
- board text added: "BATTERY"
- board text added: "DC801 Badge Team @nemus801 @pips801 @_bashNinja @admiral_potato @corfidbizna @newzie1 tazmodius @kiyoshigawa"
- board text added: "MISO"
- board text added: "MOSI"
- board text added: "RD"
- board text added: "SCK"
- board text added: "SPKR HP"
- board text added: "TE"
- board text added: "WR"
- board text removed: "AMBER"
- board text removed: "DC801 Badge Team @nemus801 @_bashNinja @admiral_potato @corfidbizna @pips801 @newzie1 tazmodius"
- board text removed: "Reset"
- board text removed: "SPKR"

Commit message: Add pads for programming jig Add 3-up panel for finals
Parts:
- added J28: UPDI, TestPoint:TestPoint_Pad_1.5x1.5mm, B.Cu at (106.5, 110.1)
- added J29: GND, TestPoint:TestPoint_Pad_1.5x1.5mm, B.Cu at (106.5, 106.5)
- added J30: USB-, TestPoint:TestPoint_Pad_1.5x1.5mm, B.Cu at (177.7, 103.8)
- added J31: USB+, TestPoint:TestPoint_Pad_1.5x1.5mm, B.Cu at (177.7, 100.1)
- added J32: VBUS, TestPoint:TestPoint_Pad_1.5x1.5mm, B.Cu at (177.7, 96.5)
- J19: value UPDI Programming -> 3.3V; footprint lib_fp:UPDI-Board-Edge -> TestPoint:TestPoint_Pad_1.5x1.5mm
- moved J19 9.90 mm to (106.5, 102.9), turned to 0 degrees
Connections:
- net /USB+ renamed USB+
- net /USB- renamed USB-
- U5 pad 14: Net-(U5-Pad14) -> +3V3
Routing:
- net GND: track 262.1 -> 244.7 mm, vias 62 -> 59
- net VBUS: track 217.0 -> 221.4 mm, vias 5 -> 7
- net USB+: track 99.3 -> 103.5 mm, vias 0 -> 2
- net USB-: track 87.1 -> 91.1 mm, vias 2 -> 4
- net +3V3: track 612.8 -> 614.5 mm, vias 25 -> 26
- net UPDI: track 36.4 -> 35.0 mm
- net SCL: track 296.0 -> 297.2 mm
- net R2: track 237.2 -> 236.1 mm
- net Net-(U1-Pad19): track 1.22 -> 2.04 mm
- net USB_CC2: track 95.5 -> 96.1 mm
- net LCD_SCK: track 69.9 -> 70.0 mm, vias 0 -> 1
- net UART_TX: vias 2 -> 3
- net UART_RX: vias 2 -> 3
- net LCD_WR: vias 0 -> 1
- net LCD_TE: vias 0 -> 1
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Other:
- board text added: "Rev 1"
- board text removed: "THIS AREA FOR FAB MARKINGS"
- board text removed: "UPDI"
