File: HW/BackBoard/purplewizard.sch (KiCad schematic (older format))
At the start: 64 parts, among them J1 3.3V, J10 SPKR-, J11 JTAG, J12 TagConnect, J13 Minibadge Expansion, J14 Battery, J15 USB_C_Receptacle_USB2.0, J16 Conn_01x50, J17 Board to Board, J18 Micro_SD_Card, J19 UPDI Programming, J2 GND, J3 UART_TX, J4 UART_RX, J5 LCD_SCK, J6 LCD_MOSI, J8 LCD_RS, J9 SPKR+, Q1 FDN360P, SW1 Power, U1 NAU8810, U2 SC189ZSKTRT, U3 BMD-340, U4 MCP73832-2-OT, U5 S25FL256S, X1 Badgelife_sao_connector_v169b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

Commit message: Backboard - Move LCD connector over .3mm for better fitment of ribbon - Fix audio chip missing exposed pad bond to ground - Remove nRESET signal from JTAG - Reuse freed pin above to run an interrupt line from the keyboard controller to the MCU to enable interrupt driven keyboard input.  Protos will have a hack-n-jump to be feature compatible - Enlarge mounting holes from 3mm to 3.2mm to allow for slightly sloppier fitments - Move traces and vias a little further away from top mounting holes as they are now being used for standoffs instead of just lanyard holes - Move vias from pads of ghosting diodes off to the side to prevent excess solder wicking - Modify UPDI programming pads to include vias for easier connection of programmer - Enlarged fiducials - Moved LCD CS from high to low - Added more breakout pads for the LCD on the back - Swapped to a PAM2305 voltage regulator - Hardwired the LCD LED to ground - Added some breakout for a couple of processor GPIO - Moved silk for speaker placement down a little - Added logo for PCBX Artboard - Remove mask over eyes
Parts:
- added C26: 10uF, Capacitor_SMD:C_0603_1608Metric, symbol Device:C
- added J20: P1.06, TestPoint:TestPoint_Pad_1.5x1.5mm, symbol Connector_Generic:Conn_01x01
- added J21: P1.05, TestPoint:TestPoint_Pad_1.5x1.5mm, symbol Connector_Generic:Conn_01x01
- added J22: LCD_MISO, TestPoint:TestPoint_Pad_1.5x1.5mm, symbol Connector_Generic:Conn_01x01
- added J23: LCD_RD, TestPoint:TestPoint_Pad_1.5x1.5mm, symbol Connector_Generic:Conn_01x01
- added J24: LCD_TE, TestPoint:TestPoint_Pad_1.5x1.5mm, symbol Connector_Generic:Conn_01x01
- added J25: MOUT, TestPoint:TestPoint_Pad_1.5x1.5mm, symbol Connector_Generic:Conn_01x01
- added J26: MIC+, TestPoint:TestPoint_Pad_1.5x1.5mm, symbol Connector_Generic:Conn_01x01
- added J27: GND, TestPoint:TestPoint_Pad_1.5x1.5mm, symbol Connector_Generic:Conn_01x01
- added J7: P1.07, TestPoint:TestPoint_Pad_1.5x1.5mm, symbol Connector_Generic:Conn_01x01
- added JP1: SolderJumper_2_Bridged, Jumper:SolderJumper-2_P1.3mm_Bridged_RoundedPad1.0x1.5mm, symbol Jumper:SolderJumper_2_Bridged
- added R17: 540k, Resistor_SMD:R_0603_1608Metric, symbol Device:R
- added R18: 120k, Resistor_SMD:R_0603_1608Metric, symbol Device:R
- FID1, FID2, FID3, FID4: footprint Fiducial:Fiducial_0.5mm_Mask1.5mm -> Fiducial:Fiducial_1mm_Mask2mm
- J8: value LCD_RS -> LCD_WR
- L1: value 1.0uH -> 4.7uH; footprint Inductor_SMD:L_Abracon_ASPI-3012S -> Inductor_SMD:L_0805_2012Metric
- U1: symbol Nuvoton:NAU8810 -> purplewizard-rescue:NAU8810-Nuvoton
- U2: value SC189ZSKTRT -> PAM2305AABADJ
- U3: footprint RIGADO_BMD-340 -> lib_fp:RIGADO_BMD-340
Connections:
- net +3V3: now also C26.2, JP1.2 (B), R17.2; no longer J16.38 (Pin_38), U2.4 (OUT)
- net GND: now also J16.11 (Pin_11), J16.12 (Pin_12), J16.13 (Pin_13), J16.14 (Pin_14), J16.15 (Pin_15), J16.16 (Pin_16), J16.17 (Pin_17), J16.18 (Pin_18), J16.19 (Pin_19), J16.2 (Pin_2), J16.20 (Pin_20), J16.21 (Pin_21), J16.22 (Pin_22), J16.23 (Pin_23), J16.24 (Pin_24), J16.25 (Pin_25), J16.26 (Pin_26), J16.27 (Pin_27), J16.28 (Pin_28), J16.29 (Pin_29), J16.3 (Pin_3), J16.30 (Pin_30), J16.31 (Pin_31), J16.32 (Pin_32), J16.38 (Pin_38), J16.4 (Pin_4), J16.5 (Pin_5), C26.1, J27.1 (Pin_1), R18.1
- net at U3.48 (P1.05): now also J21.1 (Pin_1)
- net at U3.49 (P1.06): now also J20.1 (Pin_1)
- net at U3.50 (P1.07): now also J7.1 (Pin_1)
- net at U1.13 (MOUT): now also J25.1 (Pin_1)
- net at U1.20 (MIC+): now also J26.1 (Pin_1)
- net I2S_SDIN: now reaches U1.6 (SDOUT)
- net I2S_SDIN: now also U3.12 (P0.31)
- net LCD_MISO: now reaches J16.33 (Pin_33)
- net LCD_MISO: now also J22.1 (Pin_1)
- net LCD_RD: now reaches J16.35 (Pin_35)
- net LCD_RD: now also J23.1 (Pin_1), JP1.1 (A)
- net LCD_TE: now reaches J16.39 (Pin_39)
- net LCD_TE: now also J24.1 (Pin_1)
- removed net LCD_LED: J16.2 (Pin_2), J16.3 (Pin_3), J16.4 (Pin_4), J16.5 (Pin_5), U3.12 (P0.31)
- net LCD_RS renamed LCD_WR
- removed net nRESET: J11.10 (Pin_10), J12.10 (Pin_10), U3.39 (P0.18)
- new net: R17.1, R18.2, U2.4 (OUT)
- new net KEY_INT: U3.39 (P0.18)
- no-connect marks 64 -> 35
Other:
- note added: "4 Wire Mode 1 \n(no MISO)"
- note added: "Backlight"
- note added: "Board Center"
- note added: "Board Edge"
- note added: "RD"
- moved on the sheet: C25, C4, C5, C6, FID1, FID2, FID3, FID4, J1, J10, J2, J3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

Commit message: Add pads for programming jig Add 3-up panel for finals
Parts:
- removed J19: UPDI Programming, lib_fp:UPDI-Board-Edge, symbol Connector_Generic:Conn_01x03
- added J19: 3.3V, TestPoint:TestPoint_Pad_1.5x1.5mm, symbol Connector_Generic:Conn_01x01
- added J28: UPDI, TestPoint:TestPoint_Pad_1.5x1.5mm, symbol Connector_Generic:Conn_01x01
- added J29: GND, TestPoint:TestPoint_Pad_1.5x1.5mm, symbol Connector_Generic:Conn_01x01
- added J30: USB-, TestPoint:TestPoint_Pad_1.5x1.5mm, symbol Connector_Generic:Conn_01x01
- added J31: USB+, TestPoint:TestPoint_Pad_1.5x1.5mm, symbol Connector_Generic:Conn_01x01
- added J32: VBUS, TestPoint:TestPoint_Pad_1.5x1.5mm, symbol Connector_Generic:Conn_01x01
- U1: symbol purplewizard-rescue:NAU8810-Nuvoton -> purplewizard-rescue:NAU8810-Nuvoton-purplewizard-rescue
Connections:
- net +3V3: now also U5.14 (VIO), J19.1 (Pin_1)
- net GND: now also J29.1 (Pin_1)
- net UPDI: now also J28.1 (Pin_1)
- net USB+: now also J31.1 (Pin_1)
- net USB-: now also J30.1 (Pin_1)
- net VBUS: now also J32.1 (Pin_1)
- no-connect marks 35 -> 34
Other:
- note removed: "Board Center"
- note removed: "Board Edge"
- moved on the sheet: C10, C11, D4, J1, J13, J2, J22, J23, J24, J3, J4, J5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
