File: Hardware/BackBoard/purplewizard.sch (KiCad schematic (older format))
At the start: 82 parts, among them J1 3.3V, J10 SPKR-, J11 JTAG, J12 TagConnect, J13 Minibadge Expansion, J14 Battery, J15 USB_C_Receptacle_USB2.0, J16 Conn_01x50, J17 Board to Board, J18 Micro_SD_Card, J19 3.3V, J2 GND, J20 P1.06, J21 P1.05, J22 LCD_MISO, J23 LCD_RD, J24 LCD_TE, J25 MOUT, J26 MIC+, J27 GND, J28 UPDI, J29 GND, J3 UART_TX, J30 USB-, J31 USB+, J32 VBUS, J4 UART_RX, J5 LCD_SCK, J6 LCD_MOSI, J7 P1.07, J8 LCD_WR, J9 SPKR+, Q1 FDN360P, SW1 Power, U1 NAU8810, U2 PAM2305AABADJ, U3 BMD-340, U4 MCP73832-2-OT, U5 S25FL256S, X1 Badgelife_sao_connector_v169b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

Commit message: Adding PogoProto jig Fixed upper right hole being off 3/4 of a millimeter Added some pads for USB and added some vias to help pogo pin alignment
Parts:
- added J33: SWDIO, TestPoint:TestPoint_Pad_1.5x1.5mm, symbol Connector_Generic:Conn_01x01
- added J34: SWCLK, TestPoint:TestPoint_Pad_1.5x1.5mm, symbol Connector_Generic:Conn_01x01
- added J35: SWO, TestPoint:TestPoint_Pad_1.5x1.5mm, symbol Connector_Generic:Conn_01x01
Connections:
- net SW0: now also J35.1 (Pin_1)
- net SWCLK: now also J34.1 (Pin_1)
- net SWDIO: now also J33.1 (Pin_1)
Changed lines of the file:
@@
 F 3 "~" H 10775 3680 50  0001 C CNN
 	1    10775 3680
-	-1   0    0    1
+	-1   0    0    -1
 $EndComp
 Wire Notes Line
@@
 Wire Wire Line
 	10975 5710 10975 5570
-Wire Notes Line
-	9925 6210 11825 6210
-Wire Notes Line
-	9925 610  9925 6210
-Wire Notes Line
-	11825 610  11825 6210
 Wire Wire Line
 	5485 5310 5640 5310
@@
 	-1   0    0    1
 $EndComp
+$Comp
+L Connector_Generic:Conn_01x01 J35
+U 1 1 600647D1
+P 10775 6385
+F 0 "J35" H 10855 6427 50  0000 L CNN
+F 1 "SWO" H 10855 6336 50  0000 L CNN
+F 2 "TestPoint:TestPoint_Pad_1.5x1.5mm" H 10775 6385 50  0001 C CNN
+F 3 "~" H 10775 6385 50  0001 C CNN
+	1    10775 6385
+	-1   0    0    -1
+$EndComp
+$Comp
+L Connector_Generic:Conn_01x01 J34
+U 1 1 600647DB
+P 10775 6215
+F 0 "J34" H 10854 6257 50  0000 L CNN
+F 1 "SWCLK" H 10854 6166 50  0000 L CNN
+F 2 "TestPoint:TestPoint_Pad_1.5x1.5mm" H 10775 6215 50  0001 C CNN
+F 3 "~" H 10775 6215 50  0001 C CNN
+	1    10775 6215
+	-1   0    0    -1
+$EndComp
+$Comp
+L Connector_Generic:Conn_01x01 J33
+U 1 1 600647E5
+P 10775 6050
+F 0 "J33" H 10854 6092 50  0000 L CNN
+F 1 "SWDIO" H 10854 6001 50  0000 L CNN
+F 2 "TestPoint:TestPoint_Pad_1.5x1.5mm" H 10775 6050 50  0001 C CNN
+F 3 "~" H 10775 6050 50  0001 C CNN
+	1    10775 6050
+	-1   0    0    -1
+$EndComp
+Text GLabel 10975 6215 2    50   Input ~ 10
+SWCLK
+Text GLabel 10975 6050 2    50   Input ~ 10
+SWDIO
+Text GLabel 10975 6385 2    50   Input ~ 10
+SW0
+Wire Notes Line
+	9925 6600 11825 6600
+Wire Notes Line
+	9925 610  9925 6600
+Wire Notes Line
+	11825 610  11825 6600
 $EndSCHEMATC

Commit message: Final fab files for the PCBs
Parts:
- J15: symbol Connector:USB_C_Receptacle_USB2.0 -> purplewizard-rescue:USB_C_Receptacle_USB2.0-Connector
Changed lines of the file:
@@
 	3455 3210 3685 3210
 $Comp
-L Connector:USB_C_Receptacle_USB2.0 J15
+L purplewizard-rescue:USB_C_Receptacle_USB2.0-Connector J15
 U 1 1 5EE85D2B
 P 8700 3110
