File: Hardware/BackBoard Pogo Jig/purplewizard-pogo.kicad_pcb (KiCad board)
At the start: 2 copper layers, 93 x 162 mm, 55 parts, among them J1 3.3V, J10 USB Vbus, J11 SWD, J12 TagConnect, J13 Atmel ICE UPDI, J14 USB- Select, J15 USB_C_Receptacle_USB2.0, J16 Conn_01x50, J17 Mode Select, J18 GND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

Commit message: Final fab files for the PCBs
Parts:
- added G***: LOGO, lib_fp:FrontSilk, F.Cu at (170.5, 99.6)
Other:
- board text added: "@hamster"
- board text added: "Rev 1"
