File: Hardware/BackBoard Pogo Jig/purplewizard-pogo.sch (KiCad schematic (older format))
At the start: 54 parts, among them J1 3.3V, J10 USB Vbus, J11 SWD, J12 TagConnect, J13 Atmel ICE UPDI, J14 USB- Select, J15 USB_C_Receptacle_USB2.0, J16 Conn_01x50, J17 Mode Select, J18 GND, J19 3.3V, J2 GND, J20 +3V3, J21 LCD Breakout, J22 LCD_MISO, J23 LCD_RD, J24 LCD_TE, J25 USB+ Select, J28 UPDI, J29 GND, J3 UART_TX, J30 USB-, J31 USB+, J32 VBUS, J33 3.3V, J34 GND, J35 UART_TX, J4 UART_RX, J5 LCD_SCK, J6 LCD_MOSI, J7 GND, J8 LCD_WR, J9 3V3, SW1 Power, U1 FT230XS

Commit message: Uprev to 1.1 to support current parts availability Added solderpaste to USB connector through-pins
Parts:
- C1: value 100nF -> 0.1uF
- R1, R2: value R -> 470R
Changed lines of the file:
@@
 P 6710 1980
 F 0 "R1" V 6503 1980 50  0000 C CNN
-F 1 "R" V 6594 1980 50  0000 C CNN
+F 1 "470R" V 6594 1980 50  0000 C CNN
 F 2 "Resistor_SMD:R_0603_1608Metric" V 6640 1980 50  0001 C CNN
 F 3 "~" H 6710 1980 50  0001 C CNN
@@
 P 6710 2420
 F 0 "R2" V 6503 2420 50  0000 C CNN
-F 1 "R" V 6594 2420 50  0000 C CNN
+F 1 "470R" V 6594 2420 50  0000 C CNN
 F 2 "Resistor_SMD:R_0603_1608Metric" V 6640 2420 50  0001 C CNN
 F 3 "~" H 6710 2420 50  0001 C CNN
@@
 P 1540 6325
 F 0 "C1" H 1654 6371 50  0000 L CNN
-F 1 "100nF" H 1654 6280 50  0000 L CNN
+F 1 "0.1uF" H 1654 6280 50  0000 L CNN
 F 2 "Capacitor_SMD:C_0603_1608Metric" H 1578 6175 50  0001 C CNN
 F 3 "~" H 1540 6325 50  0001 C CNN
