File: Hardware/SAOs/2022 MiniMage/MiniMageSpells.kicad_sch (KiCad schematic)
At the start: 7 parts, among them X1 Badgelife_sao_connector_v169b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

Commit message: Adding panel for SAOs
Parts:
- X1: footprint common_fp:Badgelife-Shitty-v1.69bis -> Connector_PinHeader_2.54mm:PinHeader_2x03_P2.54mm_Vertical_SMD
Changed lines of the file:
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@@
     (property "Reference" "X1" (id 0) (at 132.3848 66.7344 0))
     (property "Value" "Badgelife_sao_connector_v169bis" (id 1) (at 132.3848 69.2713 0))
-    (property "Footprint" "common_fp:Badgelife-Shitty-v1.69bis" (id 2) (at 137.4648 75.3872 90)
+    (property "Footprint" "Connector_PinHeader_2.54mm:PinHeader_2x03_P2.54mm_Vertical_SMD" (id 2) (at 137.4648 75.3872 90)
       (effects (font (size 1.27 1.27)) hide)
     )
@@
     )
     (path "/c16d125a-0138-48f1-b27b-85ca73fbe571"
-      (reference "X1") (unit 1) (value "Badgelife_sao_connector_v169bis") (footprint "common_fp:Badgelife-Shitty-v1.69bis")
+      (reference "X1") (unit 1) (value "Badgelife_sao_connector_v169bis") (footprint "Connector_PinHeader_2.54mm:PinHeader_2x03_P2.54mm_Vertical_SMD")
     )
   )
